File: hardware/logicboard/p128.sch (EAGLE design)
At the start: 59 parts, among them IC1 74LS07N, IC11 74LS153D, IC12 LTC485S, IC13 LTC485S, IC2 4066N, J1 MKR, J11 Qwiic, J12 Qwiic, J13 Qwiic, J14 Qwiic, J2 GPIO, J3 LED, J4 ALTPWR, J5 RLY, K1 G5V1, T1 2SC1815, U1 DS18B20

Commit message: First try.
Parts:
- removed D1, D2, D3: DIODE-1N4148, SparkFun-DiscreteSemi:DIODE-1N4148
- removed F1: 1.8A, fuse:TE5
- removed H1, H2: STAND-OFF, SparkFun-Hardware:STAND-OFF
- removed J1: MKR, SparkFun-Connectors:CONN_05JST
- removed J11, J12, J13, J14: Qwiic, SparkFun-Connectors:QWIIC_CONNECTORJS-1MM
- removed J2: GPIO, SparkFun-Connectors:CONN_03JST-PTH-VERT
- removed J3: LED, SparkFun-Connectors:CONN_03JST-PTH
- removed J4: ALTPWR, SparkFun-Connectors:CONN_03JST-PTH-VERT
- removed J5: RLY, SparkFun-Connectors:CONN_02JST-PTH-2
- removed JP2: MPXJMP, pinhead:PINHD-1X2
- removed JP3: RLYJMP, pinhead:PINHD-1X2
- removed JP4: PWRSEL, pinhead:PINHD-1X3
- removed JP5: GNDPIN, pinhead:PINHD-1X1
- removed K1: G5V1, relay:G5V1
- removed OK1: 6N137, optocoupler:6N137
- removed R1: 47k, resistor:R-EU_0204/5
- removed R11: 10k, rcl:R-EU_M2012
- removed R12, R13: 120, rcl:R-EU_M2012
- removed R2, R3: 1k, resistor:R-EU_0204/5
- removed R5, R6: 120, resistor:R-EU_0204/5
- removed RN1: 4.7k, resistor-net:RN04
- removed RN2: 220, resistor-dil:8R-N
- removed RN3: 10k, resistor-net:RN04
- removed SV1: (no value), con-ml:ML16LE
- removed SV2: (no value), con-ml:ML20LE
- removed T1: 2SC1815, transistor:2SC1815
- removed U1: DS18B20, SparkFun-Sensors:DS18B20
- removed V1: 5V, v-reg:78XXL
- added C14, C16: 10n, resistor:C-EU025-024X044
- added C15: 10n, rcl:C-EU025-024X044
- added IC10, IC14, IC15, IC16, IC3, IC4, IC5, IC6, IC7, IC8, IC9: 74LS595N, 74xx-us:74LS595N
- C1: value 22u -> 10n; device rcl:C-EU025-050X050 -> resistor:C-EU025-024X044
- C10, C5: value 100n -> 10n
- C11, C12, C13: device rcl:C-EUC2012 -> resistor:C-EU025-024X044
- C2: value 470n -> 10n; device rcl:C-EU050-024X044 -> resistor:C-EU025-024X044
- C3: value 1u -> 10n; device rcl:C-EU050-024X044 -> resistor:C-EU025-024X044
- C4: value 100n -> 10n; device rcl:C-EU025-024X044 -> resistor:C-EU025-024X044
- IC1: value 74LS07N -> 74LS595N; device 74xx-us:74LS07N -> 74xx-us:74LS595N
- IC11: value 74LS153D -> 74LS595N; device 74xx-us:74LS153D -> 74xx-us:74LS595N
- IC12, IC13: value LTC485S -> 74LS595N; device linear-technology:LTC485S -> 74xx-us:74LS595N
- IC2: value 4066N -> 74LS595N; device 40xx:4066N -> 74xx-us:74LS595N
- JP1: value RTC -> GNDPIN; device SparkFun-Connectors:CONN_05 -> pinhead:PINHD-1X1
Connections:
- removed net ANLG1: IC2A.A, MC1.A0, SV1-4.S
- removed net ANLG2: IC2B.A, MC1.A1, SV1-8.S
- removed net ANLG3: IC2C.A, MC1.A2, SV1-12.S
- removed net ANLG4: IC2D.A, MC1.A3, SV1-16.S
- removed net AREF: C5.1, MC1.AREF, R3.1
- removed net D7: J1.4, MC1.7
- removed net DTCT1: MC1.6, SV1-3.S
- removed net DTCT2: MC1.9, SV1-7.S
- removed net DTCT3: MC1.10, SV1-11.S
- removed net DTCT4: MC1.12, SV1-15.S
- removed net GPIO1: J2.2, MC1.5
- removed net GPIO2: J2.3, MC1.8
- removed net LED0: MC1.13, R6.2
- removed net LED0A: J3.2, R6.1
- removed net LED1: MC1.11, R5.2
- removed net LED1A: J3.3, R5.1
- removed net MIDIINSND: D3.C, OK1.A, RN2A.1
- removed net MIN: IC11A.1C1, JP2.2, OK1.VO
- removed net MIRETN: D3.A, OK1.C, SV2-8.S
- removed net MISEND: RN2A.2, SV2-7.S
- removed net MO1: IC1B.O, RN2F.1
- removed net MO1RETN: RN2F.2, SV2-14.S
- removed net MO1SEND: RN2C.2, SV2-13.S
- removed net MO2: IC1C.O, RN2G.1
- removed net MO2RETN: RN2G.2, SV2-18.S
- removed net MO2SEND: RN2D.2, SV2-17.S
- removed net MRX: IC11A.1C0, IC12.RO
- removed net MRX+: IC12.A, R12.1, SV2-9.S
- removed net MRX-: IC12.B, R12.2, SV2-11.S
- removed net MRXDTCT: IC11A.A, R11.1, SV2-10.S
- removed net MT: IC1A.O, RN2E.1
- removed net MTRETN: RN2E.2, SV2-20.S
- removed net MTSEND: RN2B.2, SV2-19.S
- removed net MTX+: IC13.A, R13.1, SV2-15.S
- removed net MTX-: IC13.B, R13.2, SV2-16.S
- removed net PDN: IC2A.C, IC2B.C, IC2C.C, IC2D.C, MC1.A4
- removed net RLY: MC1.4, R2.2
- removed net RLYDRV: R1.2, R2.1, T1.B
- removed net RLYOUT: J5.1, K12.S
- removed net RLYSNK: D2.A, K11.2, T1.C
- removed net RST: MC1.R@1, MC1.R@2, SV2-3.S
- removed net RX: IC11A.1Y, IC1A.I, JP2.1, MC1.RX, RN1.2
- removed net SCL: J1.3, J11.SCL, J12.SCL, J13.SCL, J14.SCL, JP1.4, MC1.3, RN1.4
- removed net SDA: J1.2, J11.SDA, J12.SDA, J13.SDA, J14.SDA, JP1.5, MC1.2, RN1.3
- removed net THS: MC1.A5, RN1.5, U1.DQ
- removed net TX: IC13.DI, IC1B.I, IC1C.I, MC1.TX
- removed net V5V: JP4.2, R3.2, SV1-1.S, SV1-13.S, SV1-5.S, SV1-9.S
- removed net VDD: J4.3, MC1.3V
- removed net VOUT: F1.2, JP4.1
- removed net VOUTRAW: C3.1, C4.1, D1.A, J5.2, JP3.2, K12.P, K12.P@1, V1.OUT
- new net N$6: IC11A.QH*, IC12A.SER
- new net N$7: IC13A.QH*, IC14A.SER
- new net N$9: IC15A.QH*, IC16A.SER
- new net Q1: IC1A.QA
- new net Q10: IC2A.QB
- new net Q100: IC13A.QD
- new net Q101: IC13A.QE
- new net Q102: IC13A.QF
- new net Q103: IC13A.QG
- new net Q104: IC13A.QH
- new net Q105: IC14A.QA
- new net Q106: IC14A.QB
- new net Q107: IC14A.QC
- new net Q108: IC14A.QD
- new net Q109: IC14A.QE
- new net Q11: IC2A.QC
- new net Q110: IC14A.QF
- new net Q111: IC14A.QG
- new net Q112: IC14A.QH
- new net Q113: IC15A.QA
- new net Q114: IC15A.QB
- new net Q115: IC15A.QC
- new net Q116: IC15A.QD
- new net Q117: IC15A.QE
- new net Q118: IC15A.QF
- new net Q119: IC15A.QG
- new net Q12: IC2A.QD
- new net Q120: IC15A.QH
- new net Q121: IC16A.QA
- new net Q122: IC16A.QB
- new net Q123: IC16A.QC
- new net Q124: IC16A.QD
- new net Q125: IC16A.QE
- new net Q126: IC16A.QF
- new net Q127: IC16A.QG
- new net Q128: IC16A.QH
- new net Q13: IC2A.QE
- new net Q14: IC2A.QF
- new net Q15: IC2A.QG
- new net Q16: IC2A.QH
- new net Q17: IC3A.QA
- new net Q18: IC3A.QB
- new net Q19: IC3A.QC
- new net Q2: IC1A.QB
- new net Q20: IC3A.QD
- new net Q21: IC3A.QE
- new net Q22: IC3A.QF
- new net Q23: IC3A.QG
- new net Q24: IC3A.QH
- new net Q25: IC4A.QA
- new net Q26: IC4A.QB
- new net Q27: IC4A.QC
- new net Q28: IC4A.QD
- new net Q29: IC4A.QE
- new net Q3: IC1A.QC
- new net Q30: IC4A.QF
- new net Q31: IC4A.QG
- new net Q32: IC4A.QH
- new net Q33: IC5A.QA
- new net Q34: IC5A.QB
- new net Q35: IC5A.QC
- new net Q36: IC5A.QD
- new net Q37: IC5A.QE
- new net Q38: IC5A.QF
- new net Q39: IC5A.QG
- new net Q4: IC1A.QD
- new net Q40: IC5A.QH
- new net Q41: IC6A.QA
- new net Q42: IC6A.QB
- new net Q43: IC6A.QC
- new net Q44: IC6A.QD
- new net Q45: IC6A.QE
- new net Q46: IC6A.QF
- new net Q47: IC6A.QG
- new net Q48: IC6A.QH
- new net Q49: IC7A.QA
- new net Q5: IC1A.QE
- new net Q50: IC7A.QB
- new net Q51: IC7A.QC
- new net Q52: IC7A.QD
- new net Q53: IC7A.QE
- new net Q54: IC7A.QF
- new net Q55: IC7A.QG
- new net Q56: IC7A.QH
- new net Q57: IC8A.QA
- new net Q58: IC8A.QB
- new net Q59: IC8A.QC
- new net Q6: IC1A.QF
- new net Q60: IC8A.QD
- new net Q61: IC8A.QE
- new net Q62: IC8A.QF
- new net Q63: IC8A.QG
- new net Q64: IC8A.QH
- new net Q65: IC9A.QA
- new net Q66: IC9A.QB
- new net Q67: IC9A.QC
- new net Q68: IC9A.QD
- new net Q69: IC9A.QE
- new net Q7: IC1A.QG
- new net Q70: IC9A.QF
- new net Q71: IC9A.QG
- new net Q72: IC9A.QH
- new net Q73: IC10A.QA
- new net Q74: IC10A.QB
- new net Q75: IC10A.QC
- new net Q76: IC10A.QD
- new net Q77: IC10A.QE
- new net Q78: IC10A.QF
- new net Q79: IC10A.QG
- new net Q8: IC1A.QH
- new net Q80: IC10A.QH
- new net Q81: IC11A.QA
- new net Q82: IC11A.QB
- new net Q83: IC11A.QC
- new net Q84: IC11A.QD
- new net Q85: IC11A.QE
- new net Q86: IC11A.QF
- new net Q87: IC11A.QG
- new net Q88: IC11A.QH
- new net Q89: IC12A.QA
- new net Q9: IC2A.QA
- new net Q90: IC12A.QB
- new net Q91: IC12A.QC
- new net Q92: IC12A.QD
- new net Q93: IC12A.QE
- new net Q94: IC12A.QF
- new net Q95: IC12A.QG
- new net Q96: IC12A.QH
- new net Q97: IC13A.QA
- new net Q98: IC13A.QB
- new net Q99: IC13A.QC
- new net RCLK: IC10A.RCK, IC11A.RCK, IC12A.RCK, IC13A.RCK, IC14A.RCK, IC15A.RCK, IC16A.RCK, IC1A.RCK, IC2A.RCK, IC3A.RCK, IC4A.RCK, IC5A.RCK, IC6A.RCK, IC7A.RCK, IC8A.RCK, IC9A.RCK, MC1.4
- new net SER1: IC1A.SER, MC1.5
- new net SER2: IC3A.SER, MC1.6
- new net SER3: IC5A.SER, MC1.7
- new net SER4: IC7A.SER, MC1.8
- new net SER5: IC9A.SER, MC1.9
- new net SER6: IC11A.SER, MC1.10
- new net SER7: IC13A.SER, MC1.11
- new net SER8: IC15A.SER, MC1.12
- new net SRCLK: IC10A.SCK, IC11A.SCK, IC12A.SCK, IC13A.SCK, IC14A.SCK, IC15A.SCK, IC16A.SCK, IC1A.SCK, IC2A.SCK, IC3A.SCK, IC4A.SCK, IC5A.SCK, IC6A.SCK, IC7A.SCK, IC8A.SCK, IC9A.SCK, MC1.3
- new net SRCLR: IC10A.SCL, IC11A.SCL, IC12A.SCL, IC13A.SCL, IC14A.SCL, IC15A.SCL, IC16A.SCL, IC1A.SCL, IC2A.SCL, IC3A.SCL, IC4A.SCL, IC5A.SCL, IC6A.SCL, IC7A.SCL, IC8A.SCL, IC9A.SCL, MC1.2
- net GND: now also C14.2, C15.2, C16.2, IC10A.G, IC11A.G, IC12A.G, IC13A.G, IC14A.G, IC15A.G, IC16A.G, IC1A.G, IC2A.G, IC3A.G, IC4A.G, IC5A.G, IC6A.G, IC7A.G, IC8A.G, IC9A.G, JP1.1; no longer IC11A.1C2, IC11A.1C3, IC11A.1G, IC11A.2C0, IC11A.2C1, IC11A.2C2, IC11A.2C3, IC11A.2G, IC11A.B, IC12.!RE, IC12.DE, IC12.DI, IC12.GND, IC13.GND, IC1D.I, IC1E.I, IC1F.I, IC2P.VSS, J1.1, J11.GND, J12.GND, J13.GND, J14.GND, J2.1, J3.1, J4.2, JP1.2, JP5.1, OK1.GND, R1.1, RN3.1, SV1-10.S, SV1-14.S, SV1-2.S, SV1-6.S, SV2-12.S, SV2-2.S, SV2-4.S, SV2-6.S, T1.E, U1.GND, V1.GND
- net N$1: now also IC1A.QH*, IC2A.SER; no longer IC2D.B, RN3.2
- net N$2: now also IC3A.QH*, IC4A.SER; no longer IC2C.B, RN3.3
- net N$3: now also IC5A.QH*, IC6A.SER; no longer IC2B.B, RN3.4
- net N$4: now also IC7A.QH*, IC8A.SER; no longer F1.1, JP3.1, K12.O
- net N$5: now also IC10A.SER, IC9A.QH*; no longer IC2A.B, RN3.5
- net VCC: now also C1.1, C14.1, C15.1, C16.1, C2.1, C3.1, C4.1, C5.1; no longer D2.C, IC12.VCC, IC13.!RE, IC13.DE, IC13.VCC, IC2P.VDD, J1.5, J11.VCC, J12.VCC, J13.VCC, J14.VCC, JP1.1, JP4.3, K11.1, OK1.VCC, OK1.VE, R11.2, RN1.1, RN2B.1, RN2C.1, RN2D.1, U1.VDD
- net VIN: no longer C1.1, C2.1, D1.C, J4.1, SV2-1.S, V1.IN
Other:
- note added: "Pineapple 128"
- note removed: "Pineapple II 2.0.3"
- moved on the sheet: C1, C10, C11, C12, C13, C2, C3, C4, C5, C6, C7, C8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

Commit message: Changing PCB size.
Parts:
- added C17: (no value), rcl:C-EU025-050X050
- added C18, C19: (no value), rcl:C-EU050-024X044
- added C20: (no value), rcl:C-EU025-024X044
- added D1: 1N5817-B, diode:1N5817-B
- added IC17: (no value), v-reg:78MXXS
- added J1: (no value), Seeed-Connector:JACK-DC-005'DC-005'
Connections:
- removed net VIN: MC1.9V
- new net N$8: C17.1, C18.1, D1.C, IC17.IN, J1.+
- net GND: now also C17.2, C18.2, C19.2, C20.2, IC17.GND, J1.-, J1.CDN
- net VCC: now also C19.1, C20.1, D1.A, IC17.OUT
Other:
- moved on the sheet: JP1
