File: hardware/logicboard/p128.brd (EAGLE design)
At the start: 72 x 72 mm, 59 parts, among them IC1 74LS07N, IC11 74LS153D, IC12 LTC485S, IC13 LTC485S, IC2 4066N, J1 MKR, J11 Qwiic, J12 Qwiic, J13 Qwiic, J14 Qwiic, J2 GPIO, J3 LED, J4 ALTPWR, J5 RLY, K1 G5V1, T1 2SC1815, U1 DS18B20

Commit message: First try.
Parts:
- removed D1, D2, D3: (no value), SparkFun-DiscreteSemi:DIODE-1N4148
- removed F1: 1.8A, fuse:TE5
- removed H1, H2: STAND-OFF, SparkFun-Hardware:STAND-OFF
- removed J1: MKR, SparkFun-Connectors:JST-5-PTH
- removed J11, J12, J13, J14: Qwiic, SparkFun-Connectors:1X04_1MM_RA
- removed J2: GPIO, SparkFun-Connectors:JST-3-PTH-VERT
- removed J3: LED, SparkFun-Connectors:JST-3-PTH
- removed J4: ALTPWR, SparkFun-Connectors:JST-3-PTH-VERT
- removed J5: RLY, SparkFun-Connectors:JST-2-PTH
- removed JP2: MPXJMP, pinhead:1X02
- removed JP3: RLYJMP, pinhead:1X02
- removed JP4: PWRSEL, pinhead:1X03
- removed JP5: GNDPIN, pinhead:1X01
- removed K1: G5V1, relay:G5V1
- removed OK1: 6N137, optocoupler:DIL08
- removed R1: 47k, resistor:0204/5
- removed R11: 10k, rcl:M2012
- removed R12, R13: 120, rcl:M2012
- removed R2, R3: 1k, resistor:0204/5
- removed R5, R6: 120, resistor:0204/5
- removed RN1: 4.7k, resistor-net:RN-5
- removed RN2: 220, resistor-dil:DIL16
- removed RN3: 10k, resistor-net:RN-5
- removed SV1: (no value), con-ml:ML16L
- removed SV2: (no value), con-ml:ML20L
- removed T1: 2SC1815, transistor:TO92-ECB
- removed U1: DS18B20, SparkFun-Sensors:TO-92-AMMO
- removed V1: 5V, v-reg:78XXL
- added C14, C16: 10n, resistor:C025-024X044
- added C15: 10n, rcl:C025-024X044
- added IC10, IC14, IC15, IC16, IC3, IC4, IC5, IC6, IC7, IC8, IC9: 74LS595N, 74xx-us:DIL16
- C1: value 22u -> 10n; device rcl:C025-050X050 -> resistor:C025-024X044
- C10, C5: value 100n -> 10n
- C11, C12, C13: device rcl:C2012 -> resistor:C025-024X044
- C2: value 470n -> 10n; device rcl:C050-024X044 -> resistor:C025-024X044
- C3: value 1u -> 10n; device rcl:C050-024X044 -> resistor:C025-024X044
- C4: value 100n -> 10n; device rcl:C025-024X044 -> resistor:C025-024X044
- IC1: value 74LS07N -> 74LS595N; device 74xx-us:DIL14 -> 74xx-us:DIL16
- IC11: value 74LS153D -> 74LS595N; device 74xx-us:SO16 -> 74xx-us:DIL16
- IC12, IC13: value LTC485S -> 74LS595N; device linear-technology:SOIC8 -> 74xx-us:DIL16
- IC2: value 4066N -> 74LS595N; device 40xx:DIL14 -> 74xx-us:DIL16
- JP1: value RTC -> GNDPIN; device SparkFun-Connectors:1X05 -> pinhead:1X01
- moved C8 252.7 mm to (6.00, -189.0), turned to 0 degrees
- moved C9 245.4 mm to (1.00, -196.0), turned to 0 degrees
- moved C13 244.3 mm to (11.0, -203.0), flipped to the top
- moved C7 234.3 mm to (1.00, -189.0)
- moved C12 226.0 mm to (6.00, -203.0), flipped to the top
- moved C10 223.3 mm to (1.00, -182.0)
- moved C11 212.9 mm to (1.00, -203.0), flipped to the top
- moved IC13 186.7 mm to (11.0, -140.0), flipped to the top, turned to 0 degrees
- moved C6 186.5 mm to (6.00, -182.0)
- moved IC12 157.0 mm to (11.0, -129.0), flipped to the top, turned to 0 degrees
- moved IC11 134.3 mm to (11.0, -118.0), flipped to the top, turned to 0 degrees
- moved IC1 76.0 mm to (11.0, -8.00), turned to 0 degrees
- moved IC2 56.7 mm to (11.0, -19.0), turned to 0 degrees
- moved C3 53.3 mm to (43.0, 61.0), turned to 270 degrees
- moved C2 45.8 mm to (12.0, 45.0)
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Connections:
- removed net ANLG1: IC2.1, MC1.P$31, SV1.4
- removed net ANLG2: IC2.4, MC1.P$30, SV1.8
- removed net ANLG3: IC2.8, MC1.P$29, SV1.12
- removed net ANLG4: IC2.11, MC1.P$28, SV1.16
- removed net AREF: C5.1, MC1.P$32, R3.1
- removed net D7: J1.4, MC1.P$6
- removed net DTCT1: MC1.P$7, SV1.3
- removed net DTCT2: MC1.P$4, SV1.7
- removed net DTCT3: MC1.P$3, SV1.11
- removed net DTCT4: MC1.P$1, SV1.15
- removed net GPIO1: J2.2, MC1.P$8
- removed net GPIO2: J2.3, MC1.P$5
- removed net LED0: MC1.P$34, R6.2
- removed net LED0A: J3.2, R6.1
- removed net LED1: MC1.P$2, R5.2
- removed net LED1A: J3.3, R5.1
- removed net MIDIINSND: D3.C, OK1.2, RN2.1
- removed net MIN: IC11.5, JP2.2, OK1.6
- removed net MIRETN: D3.A, OK1.3, SV2.8
- removed net MISEND: RN2.16, SV2.7
- removed net MO1: IC1.4, RN2.6
- removed net MO1RETN: RN2.11, SV2.14
- removed net MO1SEND: RN2.14, SV2.13
- removed net MO2: IC1.6, RN2.7
- removed net MO2RETN: RN2.10, SV2.18
- removed net MO2SEND: RN2.13, SV2.17
- removed net MRX: IC11.6, IC12.1
- removed net MRX+: IC12.6, R12.1, SV2.9
- removed net MRX-: IC12.7, R12.2, SV2.11
- removed net MRXDTCT: IC11.14, R11.1, SV2.10
- removed net MT: IC1.2, RN2.5
- removed net MTRETN: RN2.12, SV2.20
- removed net MTSEND: RN2.15, SV2.19
- removed net MTX+: IC13.6, R13.1, SV2.15
- removed net MTX-: IC13.7, R13.2, SV2.16
- removed net PDN: IC2.12, IC2.13, IC2.5, IC2.6, MC1.P$27
- removed net RLY: MC1.P$9, R2.2
- removed net RLYDRV: R1.2, R2.1, T1.B
- removed net RLYOUT: J5.1, K1.10
- removed net RLYSNK: D2.A, K1.9, T1.C
- removed net RST: MC1.P$13, MC1.P$22, SV2.3
- removed net RX: IC1.1, IC11.7, JP2.1, MC1.P$14, RN1.2
- removed net SCL: J1.3, J11.4, J12.4, J13.4, J14.4, JP1.4, MC1.P$10, RN1.4
- removed net SDA: J1.2, J11.3, J12.3, J13.3, J14.3, JP1.5, MC1.P$11, RN1.3
- removed net THS: MC1.P$26, RN1.5, U1.2
- removed net TX: IC1.3, IC1.5, IC13.4, MC1.P$15
- removed net V5V: JP4.2, R3.2, SV1.1, SV1.13, SV1.5, SV1.9
- removed net VDD: J4.3, MC1.P$33
- removed net VOUT: F1.2, JP4.1
- removed net VOUTRAW: C3.1, C4.1, D1.A, J5.2, JP3.2, K1.5, K1.6, V1.OUT
- new net N$6: IC11.9, IC12.14
- new net N$7: IC13.9, IC14.14
- new net N$9: IC15.9, IC16.14
- new net Q1: IC1.15
- new net Q10: IC2.1
- new net Q100: IC13.3
- new net Q101: IC13.4
- new net Q102: IC13.5
- new net Q103: IC13.6
- new net Q104: IC13.7
- new net Q105: IC14.15
- new net Q106: IC14.1
- new net Q107: IC14.2
- new net Q108: IC14.3
- new net Q109: IC14.4
- new net Q11: IC2.2
- new net Q110: IC14.5
- new net Q111: IC14.6
- new net Q112: IC14.7
- new net Q113: IC15.15
- new net Q114: IC15.1
- new net Q115: IC15.2
- new net Q116: IC15.3
- new net Q117: IC15.4
- new net Q118: IC15.5
- new net Q119: IC15.6
- new net Q12: IC2.3
- new net Q120: IC15.7
- new net Q121: IC16.15
- new net Q122: IC16.1
- new net Q123: IC16.2
- new net Q124: IC16.3
- new net Q125: IC16.4
- new net Q126: IC16.5
- new net Q127: IC16.6
- new net Q128: IC16.7
- new net Q13: IC2.4
- new net Q14: IC2.5
- new net Q15: IC2.6
- new net Q16: IC2.7
- new net Q17: IC3.15
- new net Q18: IC3.1
- new net Q19: IC3.2
- new net Q2: IC1.1
- new net Q20: IC3.3
- new net Q21: IC3.4
- new net Q22: IC3.5
- new net Q23: IC3.6
- new net Q24: IC3.7
- new net Q25: IC4.15
- new net Q26: IC4.1
- new net Q27: IC4.2
- new net Q28: IC4.3
- new net Q29: IC4.4
- new net Q3: IC1.2
- new net Q30: IC4.5
- new net Q31: IC4.6
- new net Q32: IC4.7
- new net Q33: IC5.15
- new net Q34: IC5.1
- new net Q35: IC5.2
- new net Q36: IC5.3
- new net Q37: IC5.4
- new net Q38: IC5.5
- new net Q39: IC5.6
- new net Q4: IC1.3
- new net Q40: IC5.7
- new net Q41: IC6.15
- new net Q42: IC6.1
- new net Q43: IC6.2
- new net Q44: IC6.3
- new net Q45: IC6.4
- new net Q46: IC6.5
- new net Q47: IC6.6
- new net Q48: IC6.7
- new net Q49: IC7.15
- new net Q5: IC1.4
- new net Q50: IC7.1
- new net Q51: IC7.2
- new net Q52: IC7.3
- new net Q53: IC7.4
- new net Q54: IC7.5
- new net Q55: IC7.6
- new net Q56: IC7.7
- new net Q57: IC8.15
- new net Q58: IC8.1
- new net Q59: IC8.2
- new net Q6: IC1.5
- new net Q60: IC8.3
- new net Q61: IC8.4
- new net Q62: IC8.5
- new net Q63: IC8.6
- new net Q64: IC8.7
- new net Q65: IC9.15
- new net Q66: IC9.1
- new net Q67: IC9.2
- new net Q68: IC9.3
- new net Q69: IC9.4
- new net Q7: IC1.6
- new net Q70: IC9.5
- new net Q71: IC9.6
- new net Q72: IC9.7
- new net Q73: IC10.15
- new net Q74: IC10.1
- new net Q75: IC10.2
- new net Q76: IC10.3
- new net Q77: IC10.4
- new net Q78: IC10.5
- new net Q79: IC10.6
- new net Q8: IC1.7
- new net Q80: IC10.7
- new net Q81: IC11.15
- new net Q82: IC11.1
- new net Q83: IC11.2
- new net Q84: IC11.3
- new net Q85: IC11.4
- new net Q86: IC11.5
- new net Q87: IC11.6
- new net Q88: IC11.7
- new net Q89: IC12.15
- new net Q9: IC2.15
- new net Q90: IC12.1
- new net Q91: IC12.2
- new net Q92: IC12.3
- new net Q93: IC12.4
- new net Q94: IC12.5
- new net Q95: IC12.6
- new net Q96: IC12.7
- new net Q97: IC13.15
- new net Q98: IC13.1
- new net Q99: IC13.2
- new net RCLK: IC1.12, IC10.12, IC11.12, IC12.12, IC13.12, IC14.12, IC15.12, IC16.12, IC2.12, IC3.12, IC4.12, IC5.12, IC6.12, IC7.12, IC8.12, IC9.12, MC1.P$9
- new net SER1: IC1.14, MC1.P$8
- new net SER2: IC3.14, MC1.P$7
- new net SER3: IC5.14, MC1.P$6
- new net SER4: IC7.14, MC1.P$5
- new net SER5: IC9.14, MC1.P$4
- new net SER6: IC11.14, MC1.P$3
- new net SER7: IC13.14, MC1.P$2
- new net SER8: IC15.14, MC1.P$1
- new net SRCLK: IC1.11, IC10.11, IC11.11, IC12.11, IC13.11, IC14.11, IC15.11, IC16.11, IC2.11, IC3.11, IC4.11, IC5.11, IC6.11, IC7.11, IC8.11, IC9.11, MC1.P$10
- new net SRCLR: IC1.10, IC10.10, IC11.10, IC12.10, IC13.10, IC14.10, IC15.10, IC16.10, IC2.10, IC3.10, IC4.10, IC5.10, IC6.10, IC7.10, IC8.10, IC9.10, MC1.P$11
- net GND: now also C14.2, C15.2, C16.2, IC1.8, IC10.13, IC10.8, IC12.13, IC12.8, IC13.13, IC13.8, IC14.13, IC14.8, IC15.13, IC15.8, IC16.13, IC16.8, IC2.13, IC2.8, IC3.13, IC3.8, IC4.13, IC4.8, IC5.13, IC5.8, IC6.13, IC6.8, IC7.13, IC7.8, IC8.13, IC8.8, IC9.13, IC9.8, JP1.1; no longer IC1.11, IC1.7, IC1.9, IC11.1, IC11.10, IC11.11, IC11.12, IC11.15, IC11.2, IC11.3, IC11.4, IC12.2, IC12.3, IC12.4, IC12.5, IC13.5, IC2.7, J1.1, J11.1, J12.1, J13.1, J14.1, J2.1, J3.1, J4.2, JP1.2, JP5.1, OK1.5, R1.1, RN3.1, SV1.10, SV1.14, SV1.2, SV1.6, SV2.12, SV2.2, SV2.4, SV2.6, T1.E, U1.1, V1.GND
- net N$1: now also IC1.9, IC2.14; no longer IC2.10, RN3.2
- net N$2: now also IC3.9, IC4.14; no longer IC2.9, RN3.3
- net N$3: now also IC5.9, IC6.14; no longer IC2.3, RN3.4
- net N$4: now also IC7.9, IC8.14; no longer F1.1, JP3.1, K1.1
- net N$5: now also IC10.14, IC9.9; no longer IC2.2, RN3.5
- net VCC: now also C1.1, C14.1, C15.1, C16.1, C2.1, C3.1, C4.1, C5.1, IC1.16, IC10.16, IC12.16, IC13.16, IC14.16, IC15.16, IC16.16, IC2.16, IC3.16, IC4.16, IC5.16, IC6.16, IC7.16, IC8.16, IC9.16; no longer D2.C, IC1.14, IC12.8, IC13.2, IC13.3, IC13.8, IC2.14, J1.5, J11.2, J12.2, J13.2, J14.2, JP1.1, JP4.3, K1.2, OK1.7, OK1.8, R11.2, RN1.1, RN2.2, RN2.3, RN2.4, U1.3
- net VIN: no longer C1.1, C2.1, D1.C, J4.1, SV2.1, V1.IN
Routing:
- net GND: track 424.1 -> 135.8 mm, vias 8 -> 6
- net SDA: track 176.9 -> 0.00 mm, vias 3 -> 0
- net SCL: track 159.1 -> 0.00 mm, vias 5 -> 0
- net VOUTRAW: track 146.9 -> 0.00 mm
- net VCC: track 350.9 -> 204.8 mm, vias 7 -> 5
- net RX: track 113.0 -> 0.00 mm, vias 4 -> 0
- net LED0A: track 110.8 -> 0.00 mm
- net VIN: track 133.7 -> 23.7 mm
- net MTX+: track 98.6 -> 0.00 mm
- net SRCLR: track 0.00 -> 92.0 mm, vias 0 -> 1
- net VOUT: track 91.5 -> 0.00 mm, vias 2 -> 0
- net MIRETN: track 90.5 -> 0.00 mm
- net LED1A: track 89.4 -> 0.00 mm
- net MIN: track 88.5 -> 0.00 mm, vias 2 -> 0
- net SRCLK: track 0.00 -> 75.3 mm, vias 0 -> 1
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
Commit message: Changing PCB size.
Parts:
- added C17: (no value), rcl:C025-050X050
- added C18, C19: (no value), rcl:C050-024X044
- added C20: (no value), rcl:C025-024X044
- added D1: 1N5817-B, diode:DO41-7.6
- added IC17: (no value), v-reg:78MXXS
- added J1: (no value), Seeed-Connector:3P-L14.2*W11.0*H9.0MM
- moved C10 253.6 mm to (29.0, 70.0)
- moved C11 253.6 mm to (29.0, 49.0)
- moved C12 253.6 mm to (34.0, 49.0)
- moved C13 253.6 mm to (39.0, 49.0)
- moved C14 253.6 mm to (29.0, 42.0)
- moved C15 253.6 mm to (34.0, 42.0)
- moved C16 253.6 mm to (39.0, 42.0)
- moved C6 253.6 mm to (34.0, 70.0)
- moved C7 253.6 mm to (29.0, 63.0)
- moved C8 253.6 mm to (34.0, 63.0)
- moved C9 253.6 mm to (29.0, 56.0)
- moved IC13 221.2 mm to (94.0, 65.0)
- moved IC14 219.8 mm to (100.0, 50.0)
- moved IC15 217.5 mm to (101.0, 36.0)
- moved IC16 212.4 mm to (104.0, 18.0)
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Connections:
- removed net VIN: MC1.P$20
- new net N$8: C17.1, C18.1, D1.C, IC17.IN, J1.+
- net GND: now also C17.2, C18.2, C19.2, C20.2, IC17.GND, J1.-1, J1.-2
- net VCC: now also C19.1, C20.1, D1.A, IC17.OUT
Routing:
- net VCC: track 204.8 -> 0.00 mm, vias 5 -> 0
- net GND: track 135.8 -> 0.00 mm, vias 6 -> 0
- net SRCLR: track 92.0 -> 0.00 mm, vias 1 -> 0
- net SRCLK: track 75.3 -> 0.00 mm, vias 1 -> 0
- net SER5: track 43.3 -> 0.00 mm
- net SER6: track 40.9 -> 0.00 mm
- net SER1: track 40.4 -> 0.00 mm, vias 1 -> 0
- net RCLK: track 38.4 -> 0.00 mm
- net SER2: track 38.0 -> 0.00 mm, vias 1 -> 0
- net SER8: track 37.2 -> 0.00 mm
- net SER4: track 32.0 -> 0.00 mm
- net SER3: track 30.0 -> 0.00 mm
- net VIN: track 23.7 -> 0.00 mm, vias 2 -> 0
- net SER7: track 12.2 -> 0.00 mm
- removed copper zone on layer 1, net GND
- removed copper zone on layer 16, net GND
Other:
- board size 72 x 72 mm -> 100 x 80 mm
- board text added: "Pineapple 128"
- board text removed: "4066B"
- board text removed: "5V"
- board text removed: "ARD"
- board text removed: "NC"
- board text removed: "Pineapple II"
- board text removed: "REG"
- board text removed: "RTC1"
- board text removed: "SC"
- board text removed: "SD"
- board text removed: "SparkFun Real Time Clock Module (12708)"

Commit message: Packing in 80x80mm...
Parts:
- moved JP1 84.2 mm to (4.00, 11.0)
- moved C6 65.8 mm to (15.0, 7.00)
- moved IC5 64.1 mm to (32.0, 19.0)
- moved IC6 61.3 mm to (32.0, 7.00)
- moved IC8 61.0 mm to (56.0, 55.0)
- moved IC7 56.6 mm to (56.0, 67.0)
- moved C13 48.6 mm to (10.0, 10.0)
- moved LOGO1 44.8 mm to (14.0, 75.0)
- moved IC12 41.0 mm to (56.0, 7.00)
- moved U$1 40.3 mm to (41.0, 73.5)
- moved IC11 39.5 mm to (56.0, 19.0)
- moved C4 38.3 mm to (14.0, 39.0)
- moved IC10 38.3 mm to (56.0, 31.0)
- moved C10 37.2 mm to (10.0, 38.0)
- moved IC9 36.1 mm to (56.0, 43.0)
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Other:
- board size 100 x 80 mm -> 80 x 80 mm
- board text removed: "74LS07"
- board text removed: "Arduino Micro"
- board text removed: "Close Here"
- board text removed: "MC1"
- board text removed: "TLP552"
