File: hardware/logicboard/p128.brd (EAGLE design)
At the start: 95 x 72 mm, 36 parts, among them IC1 74LS595N, IC2 74LS595N, IC3 74LS595N, IC4 74LS595N, IC5 74LS595N, IC6 74LS595N, IC7 74LS595N, IC8 74LS595N, J9 DC5V

Commit message: Fine tuning.
Parts:
- moved J2 3.51 mm to (19.6, 7.54)
- moved J1 3.51 mm to (19.6, 5.00)
- moved J3 3.51 mm to (19.6, 12.6)
- moved J4 3.51 mm to (19.6, 15.2)
- moved JP1 3.00 mm to (14.0, 5.00)
- moved U$1 2.00 mm to (85.0, 12.0)
- moved J6 1.41 mm to (52.6, 7.54)
- moved J5 1.41 mm to (52.6, 5.00)
- moved J7 1.41 mm to (52.6, 12.6)
- moved J8 1.41 mm to (52.6, 15.2)
Routing:
- net GND: track 542.0 -> 493.0 mm, vias 8 -> 4
- net N604: track 68.0 -> 33.2 mm, vias 1 -> 0
- net CLR: track 265.7 -> 296.9 mm, vias 10 -> 9
- net N703: track 94.4 -> 64.9 mm
- net XOUT5: track 102.5 -> 74.1 mm, vias 2 -> 5
- net N505: track 43.1 -> 70.8 mm, vias 0 -> 1
- net SCLK: track 294.2 -> 278.0 mm, vias 6 -> 7
- net N702: track 59.9 -> 44.0 mm, vias 2 -> 3
- net N802: track 48.1 -> 63.8 mm
- net VCC: track 222.3 -> 237.9 mm, vias 1 -> 2
- net XOUT2: track 90.2 -> 105.7 mm, vias 4 -> 3
- net N804: track 41.4 -> 53.4 mm
- net SIN8: track 62.9 -> 74.7 mm
- net N403: track 27.3 -> 39.1 mm
- net RCLK: track 306.4 -> 317.7 mm, vias 10 -> 6
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- added copper zone on layer 1, net GND
- added copper zone on layer 16, net GND
Other:
- board text added: "For Necobit DT-8 R3"
- board text added: "INPUT"
- board text added: "K"
