File: hardware/logicboard/p128.brd (EAGLE design)
At the start: 95 x 72 mm, 36 parts, among them IC1 74LS595N, IC2 74LS595N, IC3 74LS595N, IC4 74LS595N, IC5 74LS595N, IC6 74LS595N, IC7 74LS595N, IC8 74LS595N, J9 DC5V

Commit message: Fine fine tuning.
Parts:
- turned DZ1 to 0 degrees
Routing:
- net RCLK: track 317.7 -> 226.2 mm, vias 6 -> 9
- net N605: track 30.4 -> 81.6 mm
- net N603: track 33.4 -> 83.5 mm, vias 0 -> 3
- net N204: track 42.5 -> 79.6 mm, vias 3 -> 0
- net N$10: track 6.15 -> 29.0 mm
- net N$1: track 37.8 -> 15.2 mm
- net XOUT1: track 97.9 -> 118.6 mm, vias 1 -> 0
- net N$9: track 7.88 -> 27.5 mm
- net SIN1: track 105.8 -> 87.6 mm
- net N$2: track 34.5 -> 16.7 mm, vias 1 -> 0
- net CLR: track 296.9 -> 280.0 mm, vias 9 -> 4
- net SOUT5: track 17.3 -> 34.1 mm
- net N505: track 70.8 -> 54.4 mm
- net N$3: track 35.1 -> 19.5 mm
- net SIN4: track 74.4 -> 58.9 mm, vias 2 -> 0
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Other:
- board text added: "A"
- board text added: "C"
- board text added: "L"
- board text removed: "K"
