File: hardware/logicboard/p128control.sch (EAGLE design)
At the start: 23 parts, among them IC1 74LS158N, J2 DIN5

Commit message: SW.
Parts:
- added C2: (no value), resistor:C-EU025-024X044
- R1: value (none) -> 220
- R2, RN1: value (none) -> 10k
Connections:
- net GND: now also C2.2
- net VCC: now also C2.1
Other:
- moved on the sheet: C1
Changed lines of the file:
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@@
 <part name="OK1" library="optocoupler" library_urn="urn:adsk.eagle:library:320" deviceset="6N137" device="" package3d_urn="urn:adsk.eagle:package:21941/1"/>
 <part name="D1" library="SparkFun-DiscreteSemi" library_urn="urn:adsk.eagle:library:514" deviceset="DIODE" device="-1N4148" package3d_urn="urn:adsk.eagle:package:38452/1" value="200mA/100V/1V"/>
-<part name="R1" library="resistor" library_urn="urn:adsk.eagle:library:348" deviceset="R-EU_" device="0204/5" package3d_urn="urn:adsk.eagle:package:25955/1"/>
-<part name="R2" library="resistor" library_urn="urn:adsk.eagle:library:348" deviceset="R-EU_" device="0204/5" package3d_urn="urn:adsk.eagle:package:25955/1"/>
+<part name="R1" library="resistor" library_urn="urn:adsk.eagle:library:348" deviceset="R-EU_" device="0204/5" package3d_urn="urn:adsk.eagle:package:25955/1" value="220"/>
+<part name="R2" library="resistor" library_urn="urn:adsk.eagle:library:348" deviceset="R-EU_" device="0204/5" package3d_urn="urn:adsk.eagle:package:25955/1" value="10k"/>
 <part name="SUPPLY1" library="supply2" deviceset="GND" device=""/>
 <part name="C1" library="resistor" library_urn="urn:adsk.eagle:library:348" deviceset="C-EU" device="025-024X044" package3d_urn="urn:adsk.eagle:package:26149/1"/>
@@
 <part name="SUPPLY2" library="supply2" deviceset="GND" device=""/>
 <part name="IC1" library="74xx-us" library_urn="urn:adsk.eagle:library:88" deviceset="74*158" device="N" package3d_urn="urn:adsk.eagle:package:922/2" technology="LS"/>
-<part name="RN1" library="resistor-dil" library_urn="urn:adsk.eagle:library:342" deviceset="8R-N" device="" package3d_urn="urn:adsk.eagle:package:922/2"/>
+<part name="RN1" library="resistor-dil" library_urn="urn:adsk.eagle:library:342" deviceset="8R-N" device="" package3d_urn="urn:adsk.eagle:package:922/2" value="10k"/>
 <part name="P+4" library="supply1" library_urn="urn:adsk.eagle:library:371" deviceset="VCC" device=""/>
 <part name="SUPPLY3" library="supply2" deviceset="GND" device=""/>
@@
 <part name="SUPPLY4" library="supply2" deviceset="GND" device=""/>
 <part name="SUPPLY5" library="supply2" deviceset="GND" device=""/>
+<part name="C2" library="resistor" library_urn="urn:adsk.eagle:library:348" deviceset="C-EU" device="025-024X044" package3d_urn="urn:adsk.eagle:package:26149/1"/>
+<part name="P+5" library="supply1" library_urn="urn:adsk.eagle:library:371" deviceset="VCC" device=""/>
+<part name="SUPPLY6" library="supply2" deviceset="GND" device=""/>
 </parts>
 <sheets>
@@
 </instance>
 <instance part="SUPPLY1" gate="GND" x="144.78" y="88.9" smashed="yes"/>
-<instance part="C1" gate="G$1" x="129.54" y="99.06" smashed="yes">
-<attribute name="NAME" x="131.064" y="99.441" size="1.778" layer="95"/>
-<attribute name="VALUE" x="131.064" y="94.361" size="1.778" layer="96"/>
+<instance part="C1" gate="G$1" x="101.6" y="17.78" smashed="yes">
+<attribute name="NAME" x="103.124" y="18.161" size="1.778" layer="95"/>
+<attribute name="VALUE" x="103.124" y="13.081" size="1.778" layer="96"/>
 </instance>
 <instance part="P+2" gate="VCC" x="144.78" y="116.84" smashed="yes">
 <attribute name="VALUE" x="142.24" y="114.3" size="1.778" layer="96" rot="R90"/>
 </instance>
-<instance part="P+3" gate="VCC" x="129.54" y="106.68" smashed="yes">
-<attribute name="VALUE" x="127" y="104.14" size="1.778" layer="96" rot="R90"/>
-</instance>
-<instance part="SUPPLY2" gate="GND" x="129.54" y="88.9" smashed="yes"/>
+<instance part="P+3" gate="VCC" x="101.6" y="25.4" smashed="yes">
+<attribute name="VALUE" x="99.06" y="22.86" size="1.778" layer="96" rot="R90"/>
+</instance>
+<instance part="SUPPLY2" gate="GND" x="101.6" y="7.62" smashed="yes"/>
 <instance part="IC1" gate="A" x="185.42" y="50.8" smashed="yes">
 <attribute name="NAME" x="177.8" y="66.675" size="1.778" layer="95"/>
@@
 <instance part="SUPPLY4" gate="GND" x="101.6" y="33.02" smashed="yes"/>
 <instance part="SUPPLY5" gate="GND" x="114.3" y="33.02" smashed="yes"/>
+<instance part="C2" gate="G$1" x="114.3" y="17.78" smashed="yes">
+<attribute name="NAME" x="115.824" y="18.161" size="1.778" layer="95"/>
+<attribute name="VALUE" x="115.824" y="13.081" size="1.778" layer="96"/>
+</instance>
+<instance part="P+5" gate="VCC" x="114.3" y="25.4" smashed="yes">
+<attribute name="VALUE" x="111.76" y="22.86" size="1.778" layer="96" rot="R90"/>
+</instance>
+<instance part="SUPPLY6" gate="GND" x="114.3" y="7.62" smashed="yes"/>
 </instances>
 <busses>
@@
 <pinref part="C1" gate="G$1" pin="2"/>
 <pinref part="SUPPLY2" gate="GND" pin="GND"/>
-<wire x1="129.54" y1="93.98" x2="129.54" y2="91.44" width="0.1524" layer="91"/>
+<wire x1="101.6" y1="12.7" x2="101.6" y2="10.16" width="0.1524" layer="91"/>
 </segment>
 <segment>
@@
 <pinref part="SUPPLY5" gate="GND" pin="GND"/>
 <wire x1="114.3" y1="38.1" x2="114.3" y2="35.56" width="0.1524" layer="91"/>
+</segment>
+<segment>
+<pinref part="C2" gate="G$1" pin="2"/>
+<pinref part="SUPPLY6" gate="GND" pin="GND"/>
+<wire x1="114.3" y1="12.7" x2="114.3" y2="10.16" width="0.1524" layer="91"/>
 </segment>
 </net>
@@
 <pinref part="P+3" gate="VCC" pin="VCC"/>
 <pinref part="C1" gate="G$1" pin="1"/>
-<wire x1="129.54" y1="104.14" x2="129.54" y2="101.6" width="0.1524" layer="91"/>
+<wire x1="101.6" y1="22.86" x2="101.6" y2="20.32" width="0.1524" layer="91"/>
 </segment>
 <segment>
@@
 <junction x="134.62" y="78.74"/>
 </segment>
+<segment>
+<pinref part="P+5" gate="VCC" pin="VCC"/>
+<pinref part="C2" gate="G$1" pin="1"/>
+<wire x1="114.3" y1="22.86" x2="114.3" y2="20.32" width="0.1524" layer="91"/>
+</segment>
 </net>

Commit message: Release candidate.
Parts:
- added JP2: (no value), pinhead:PINHD-1X6
Connections:
- new net TX: JP2.5, U$2.TX
- net GND: now also JP2.1, JP2.2
- net RX: now also JP2.4
- net VCC: now also JP2.3
Changed lines of the file:
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@@
 <part name="P+5" library="supply1" library_urn="urn:adsk.eagle:library:371" deviceset="VCC" device=""/>
 <part name="SUPPLY6" library="supply2" deviceset="GND" device=""/>
+<part name="JP2" library="pinhead" library_urn="urn:adsk.eagle:library:325" deviceset="PINHD-1X6" device="" package3d_urn="urn:adsk.eagle:package:22472/2"/>
 </parts>
 <sheets>
 <sheet>
 <plain>
-<text x="223.52" y="139.7" size="1.778" layer="94" align="bottom-center">Pineapple 128</text>
+<text x="228.6" y="15.24" size="1.778" layer="94" align="bottom-center">Pineapple 128</text>
 </plain>
 <instances>
-<instance part="LOGO1" gate="G$1" x="228.6" y="109.22" smashed="yes"/>
-<instance part="U$1" gate="G$1" x="226.06" y="147.32" smashed="yes"/>
+<instance part="LOGO1" gate="G$1" x="139.7" y="12.7" smashed="yes"/>
+<instance part="U$1" gate="G$1" x="182.88" y="2.54" smashed="yes"/>
 <instance part="JP1" gate="G$1" x="10.16" y="40.64" smashed="yes" rot="R90">
 <attribute name="NAME" x="10.16" y="45.72" size="1.778" layer="95" align="bottom-center"/>
@@
 </instance>
 <instance part="SUPPLY6" gate="GND" x="114.3" y="7.62" smashed="yes"/>
+<instance part="JP2" gate="A" x="7.62" y="66.04" smashed="yes" rot="R180">
+<attribute name="NAME" x="13.97" y="55.245" size="1.778" layer="95" rot="R180"/>
+<attribute name="VALUE" x="13.97" y="76.2" size="1.778" layer="96" rot="R180"/>
+</instance>
 </instances>
 <busses>
@@
 <pinref part="SUPPLY6" gate="GND" pin="GND"/>
 <wire x1="114.3" y1="12.7" x2="114.3" y2="10.16" width="0.1524" layer="91"/>
+</segment>
+<segment>
+<pinref part="JP2" gate="A" pin="1"/>
+<wire x1="10.16" y1="58.42" x2="15.24" y2="58.42" width="0.1524" layer="91"/>
+<label x="15.24" y="58.42" size="0.8128" layer="95" xref="yes"/>
+</segment>
+<segment>
+<pinref part="JP2" gate="A" pin="2"/>
+<wire x1="10.16" y1="60.96" x2="15.24" y2="60.96" width="0.1524" layer="91"/>
+<label x="15.24" y="60.96" size="0.8128" layer="95" xref="yes"/>
 </segment>
 </net>
@@
 <wire x1="114.3" y1="22.86" x2="114.3" y2="20.32" width="0.1524" layer="91"/>
 </segment>
+<segment>
+<pinref part="JP2" gate="A" pin="3"/>
+<wire x1="10.16" y1="63.5" x2="15.24" y2="63.5" width="0.1524" layer="91"/>
+<label x="15.24" y="63.5" size="0.8128" layer="95" xref="yes"/>
+</segment>
 </net>
 <net name="CLR" class="0">
@@
 <label x="124.46" y="129.54" size="0.8128" layer="95" xref="yes"/>
 </segment>
+<segment>
+<pinref part="JP2" gate="A" pin="4"/>
+<wire x1="10.16" y1="66.04" x2="15.24" y2="66.04" width="0.1524" layer="91"/>
+<label x="15.24" y="66.04" size="0.8128" layer="95" xref="yes"/>
+</segment>
 </net>
 <net name="SW1" class="0">
@@
 </segment>
 </net>
+<net name="TX" class="0">
+<segment>
+<pinref part="U$2" gate="G$1" pin="TX"/>
+<wire x1="119.38" y1="127" x2="124.46" y2="127" width="0.1524" layer="91"/>
+<label x="124.46" y="127" size="0.8128" layer="95" xref="yes"/>
+</segment>
+<segment>
+<pinref part="JP2" gate="A" pin="5"/>
+<wire x1="10.16" y1="68.58" x2="15.24" y2="68.58" width="0.1524" layer="91"/>
+<label x="15.24" y="68.58" size="0.8128" layer="95" xref="yes"/>
+</segment>
+</net>
