File: hardware/logicboard/p128relay.sch (EAGLE design)
At the start: 30 parts, among them IC1 74LS595N, IC2 74LS595N, K1 AQG12105, K10 AQG12105, K11 AQG12105, K12 AQG12105, K13 AQG12105, K14 AQG12105, K15 AQG12105, K16 AQG12105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

Commit message: Release candidate.
Changed lines of the file:
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@@
 <sheet>
 <plain>
-<text x="294.64" y="101.6" size="1.778" layer="94" align="bottom-center">Pineapple 128</text>
+<text x="228.6" y="15.24" size="1.778" layer="94" align="bottom-center">Pineapple 128</text>
 </plain>
 <instances>
-<instance part="LOGO1" gate="G$1" x="304.8" y="78.74" smashed="yes"/>
-<instance part="U$1" gate="G$1" x="297.18" y="111.76" smashed="yes"/>
+<instance part="LOGO1" gate="G$1" x="134.62" y="15.24" smashed="yes"/>
+<instance part="U$1" gate="G$1" x="185.42" y="5.08" smashed="yes"/>
 <instance part="J1" gate="JACK" x="12.7" y="157.48" smashed="yes">
 <attribute name="NAME" x="7.62" y="162.56" size="1.27" layer="95" ratio="10"/>
