File: hardware/logicboard/p128fet.sch (EAGLE design)
At the start: 30 parts, among them IC1 74LS595N, IC2 74LS595N, K1 AQG12105, K10 AQG12105, K11 AQG12105, K12 AQG12105, K13 AQG12105, K14 AQG12105, K15 AQG12105, K16 AQG12105, K2 AQG12105, K3 AQG12105, K4 AQG12105, K5 AQG12105, K6 AQG12105, K7 AQG12105, K8 AQG12105, K9 AQG12105

Commit message: Added FET version.
Parts:
- removed C3, C4: (no value), resistor:C-EU025-024X044
- removed K1, K10, K11, K12, K13, K14, K15, K16, K2, K3, K4, K5, K6, K7, K8, K9: AQG12105, relay:AQG12105
- removed ULN1, ULN2: (no value), SparkFun-IC-Special-Function:ULN2803DIP
- added D1, D10, D11, D12, D13, D14, D15, D16, D2, D3, D4, D5, D6, D7, D8, D9: 200mA/100V/1V, SparkFun-DiscreteSemi:DIODE-1N4148
- added Q1, Q10, Q11, Q12, Q13, Q14, Q15, Q16, Q2, Q3, Q4, Q5, Q6, Q7, Q8, Q9: 60V/32A/35mΩ, SparkFun-DiscreteSemi:MOSFET-NCH-FQP30N06L
- added RN1, RN2: 220, resistor-dil:8R-N
- added RN3, RN4: 10k, resistor-dil:8R-N
Connections:
- removed net R1: K1.K, ULN1.18
- removed net R10: K10.K, ULN2.17
- removed net R11: K11.K, ULN2.16
- removed net R12: K12.K, ULN2.15
- removed net R13: K13.K, ULN2.14
- removed net R14: K14.K, ULN2.13
- removed net R15: K15.K, ULN2.12
- removed net R16: K16.K, ULN2.11
- removed net R2: K2.K, ULN1.17
- removed net R3: K3.K, ULN1.16
- removed net R4: K4.K, ULN1.15
- removed net R5: K5.K, ULN1.14
- removed net R6: K6.K, ULN1.13
- removed net R7: K7.K, ULN1.12
- removed net R8: K8.K, ULN1.11
- removed net R9: K9.K, ULN2.18
- new net N$1: Q1.G, RN1A.2
- new net N$10: Q9.G, RN2A.2
- new net N$11: Q10.G, RN2B.2
- new net N$12: Q14.G, RN2F.2
- new net N$13: Q11.G, RN2C.2
- new net N$14: Q15.G, RN2G.2
- new net N$15: Q12.G, RN2D.2
- new net N$16: Q16.G, RN2H.2
- new net N$2: Q2.G, RN1B.2
- new net N$25: Q13.G, RN2E.2
- new net N$3: Q3.G, RN1C.2
- new net N$4: Q4.G, RN1D.2
- new net N$5: Q5.G, RN1E.2
- new net N$6: Q6.G, RN1F.2
- new net N$7: Q7.G, RN1G.2
- new net N$8: Q8.G, RN1H.2
- net +24V: now also D1.C, D10.C, D11.C, D12.C, D13.C, D14.C, D15.C, D16.C, D2.C, D3.C, D4.C, D5.C, D6.C, D7.C, D8.C, D9.C, Q1.D, Q10.D, Q11.D, Q12.D, Q13.D, Q14.D, Q15.D, Q16.D, Q2.D, Q3.D, Q4.D, Q5.D, Q6.D, Q7.D, Q8.D, Q9.D; no longer K1.DS1, K10.DS1, K11.DS1, K12.DS1, K13.DS1, K14.DS1, K15.DS1, K16.DS1, K2.DS1, K3.DS1, K4.DS1, K5.DS1, K6.DS1, K7.DS1, K8.DS1, K9.DS1
- net GND: now also RN3A.1, RN3B.1, RN3C.1, RN3D.1, RN3E.1, RN3F.1, RN3G.1, RN3H.1, RN4A.1, RN4B.1, RN4C.1, RN4D.1, RN4E.1, RN4F.1, RN4G.1, RN4H.1; no longer C3.2, C4.2, ULN1.9, ULN2.9
- net S1: now also RN1A.1, RN3A.2; no longer ULN1.1
- net S10: now also RN2B.1, RN4B.2; no longer ULN2.2
- net S11: now also RN2C.1, RN4C.2; no longer ULN2.3
- net S12: now also RN2D.1, RN4D.2; no longer ULN2.4
- net S13: now also RN2E.1, RN4E.2; no longer ULN2.5
- net S14: now also RN2F.1, RN4F.2; no longer ULN2.6
- net S15: now also RN2G.1, RN4G.2; no longer ULN2.7
- net S16: now also RN2H.1, RN4H.2; no longer ULN2.8
- net S2: now also RN1B.1, RN3B.2; no longer ULN1.2
- net S3: now also RN1C.1, RN3C.2; no longer ULN1.3
- net S4: now also RN1D.1, RN3D.2; no longer ULN1.4
- net S5: now also RN1E.1, RN3E.2; no longer ULN1.5
- net S6: now also RN1F.1, RN3F.2; no longer ULN1.6
- net S7: now also RN1G.1, RN3G.2; no longer ULN1.7
- net S8: now also RN1H.1, RN3H.2; no longer ULN1.8
- net S9: now also RN2A.1, RN4A.2; no longer ULN2.1
- net VCC: no longer C3.1, C4.1, K1.A, K10.A, K11.A, K12.A, K13.A, K14.A, K15.A, K16.A, K2.A, K3.A, K4.A, K5.A, K6.A, K7.A, K8.A, K9.A, ULN1.10, ULN2.10
- net X1: now also D1.A, Q1.S; no longer K1.DS2
- net X10: now also D10.A, Q10.S; no longer K10.DS2
- net X11: now also D11.A, Q11.S; no longer K11.DS2
- net X12: now also D12.A, Q12.S; no longer K12.DS2
- net X13: now also D13.A, Q13.S; no longer K13.DS2
- net X14: now also D14.A, Q14.S; no longer K14.DS2
- net X15: now also D15.A, Q15.S; no longer K15.DS2
- net X16: now also D16.A, Q16.S; no longer K16.DS2
- net X2: now also D2.A, Q2.S; no longer K2.DS2
- net X3: now also D3.A, Q3.S; no longer K3.DS2
- net X4: now also D4.A, Q4.S; no longer K4.DS2
- net X5: now also D5.A, Q5.S; no longer K5.DS2
- net X6: now also D6.A, Q6.S; no longer K6.DS2
- net X7: now also D7.A, Q7.S; no longer K7.DS2
- net X8: now also D8.A, Q8.S; no longer K8.DS2
- net X9: now also D9.A, Q9.S; no longer K9.DS2
Other:
- moved on the sheet: IC1, IC2
